File: 4u-simple-integrator/kicad/4u-simple-integrator.kicad_pcb (KiCad board)
At the start: 2 copper layers, 48.3 x 152.4 mm, 45 parts, among them J1 BananaJack_PanelMount, J10 I1_Main, J11 4U_Power, J2 BananaJack_PanelMount, J3 BananaJack_PanelMount, J4 BananaJack_PanelMount, J5 BananaJack_PanelMount, J6 BananaJack_PanelMount, J7 I2_Ctrl, J8 I1_Ctrl, J9 I2_Main, U1 TL074

Commit message: Refreshing kicad projects
Parts:
- C1, C2, C3, C4: footprint rumblesan-standard-parts:C_Rect_L7.0mm_W3.5mm_P5.00mm -> Rumblesan_Standard_Parts:C_Rect_L7.0mm_W3.5mm_P5.00mm
- C5, C6: footprint rumblesan-standard-parts:CP_Radial_D5.0mm_P2.00mm -> Rumblesan_Standard_Parts:CP_Radial_D5.0mm_P2.00mm
- D1, D2: footprint rumblesan-standard-parts:D_DO-41_SOD81_P10.16mm_Horizontal -> Rumblesan_Standard_Parts:D_DO-41_SOD81_P10.16mm_Horizontal
- J1, J2, J3, J4, J5, J6: footprint rumblesan-standard-parts:BananaJack_THT_JohnsonCinch_108-09 -> Rumblesan_Standard_Parts:BananaJack_THT_JohnsonCinch_108-09
- J11: footprint 4u-power:4u_Power_Molex_KK-254_P2.54mm -> 4U_Power:4u_Power_Molex_KK-254_P2.54mm
- R1, R10, R11, R12, R2, R3, R4, R5, R6, R7, R8, R9: footprint rumblesan-standard-parts:R_Axial_DIN0207_L6.3mm_D2.5mm_P10.16mm_Horizontal -> Rumblesan_Standard_Parts:R_Axial_DIN0207_L6.3mm_D2.5mm_P10.16mm_Horizontal
- RV1, RV2: footprint rumblesan-standard-parts:Potentiometer_Alpha_RD901F-40-00D_Single_Vertical -> Rumblesan_Standard_Parts:Potentiometer_Alpha_RD901F-40-00D_Single_Vertical
- U1: footprint rumblesan-standard-parts:DIP-14_W7.62mm_Socket -> Rumblesan_Standard_Parts:DIP-14_W7.62mm_Socket
