File: 4u-simple-integrator/kicad/4u-simple-integrator.kicad_sch (KiCad schematic)
At the start: 38 parts, among them J1 BananaJack_PanelMount, J10 I1_Main, J11 4U_Power, J2 BananaJack_PanelMount, J3 BananaJack_PanelMount, J4 BananaJack_PanelMount, J5 BananaJack_PanelMount, J6 BananaJack_PanelMount, J7 I2_Ctrl, J8 I1_Ctrl, J9 I2_Main, U1 TL074

Commit message: Refreshing kicad projects
Parts:
- removed C1, C2: 1nF, rumblesan-standard-parts:C_Rect_L7.0mm_W3.5mm_P5.00mm, symbol rumblesan-standard-parts:C
- removed C3, C4: 100nF, rumblesan-standard-parts:C_Rect_L7.0mm_W3.5mm_P5.00mm, symbol rumblesan-standard-parts:C
- removed C5, C6: 10uF, rumblesan-standard-parts:CP_Radial_D5.0mm_P2.00mm, symbol rumblesan-standard-parts:C_Polarized
- removed D1, D2: 1N5818, rumblesan-standard-parts:D_DO-41_SOD81_P10.16mm_Horizontal, symbol Diode:1N5818
- removed J11: 4U_Power, 4u-power:4u_Power_Molex_KK-254_P2.54mm, symbol 4U_Hardware:4U_Power
- added C1, C2: 1nF, Rumblesan_Standard_Parts:C_Rect_L7.0mm_W3.5mm_P5.00mm, symbol Rumblesan Standard Parts:C
- added C3, C4: 100nF, Rumblesan_Standard_Parts:C_Rect_L7.0mm_W3.5mm_P5.00mm, symbol Rumblesan Standard Parts:C
- added C5, C6: 10uF, Rumblesan_Standard_Parts:CP_Radial_D5.0mm_P2.00mm, symbol Rumblesan Standard Parts:C_Polarized
- added D1, D2: 1N5818, Rumblesan_Standard_Parts:D_DO-41_SOD81_P10.16mm_Horizontal, symbol Device:D_Schottky
- added J11: 4U_Power, 4U_Power:4u_Power_Molex_KK-254_P2.54mm, symbol 4U_Power:4U_Power
- J1, J2, J3, J4, J5, J6: footprint rumblesan-standard-parts:BananaJack_THT_JohnsonCinch_108-09 -> Rumblesan_Standard_Parts:BananaJack_THT_JohnsonCinch_108-09; symbol BananaJacks:Banana Socket PanelMount -> Banana_Jacks:Banana_Socket_PanelMount
- J10, J9: symbol Connector:Conn_01x04_Male -> Connector:Conn_01x04_Pin
- J7, J8: symbol Connector:Conn_01x04_Female -> Connector:Conn_01x04_Socket
- R1, R10, R11, R12, R2, R3, R4, R5, R6, R7, R8, R9: footprint rumblesan-standard-parts:R_Axial_DIN0207_L6.3mm_D2.5mm_P10.16mm_Horizontal -> Rumblesan_Standard_Parts:R_Axial_DIN0207_L6.3mm_D2.5mm_P10.16mm_Horizontal; symbol rumblesan-standard-parts:R -> Rumblesan Standard Parts:R
- RV1, RV2: footprint rumblesan-standard-parts:Potentiometer_Alpha_RD901F-40-00D_Single_Vertical -> Rumblesan_Standard_Parts:Potentiometer_Alpha_RD901F-40-00D_Single_Vertical
- U1: footprint rumblesan-standard-parts:DIP-14_W7.62mm_Socket -> Rumblesan_Standard_Parts:DIP-14_W7.62mm_Socket
Connections:
- net +12V: now also C3.1, C5.1, D1.1 (K)
- net -12V: now also C4.2, C6.2, D2.2 (A)
- net GND: now also C3.2, C4.1, C5.2, C6.1, J11.2 (GND), J11.3 (GND)
- net at R3.1, R6.1, R8.2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: now also C2.2
- net at R4.1, R5.1, R7.2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: now also C1.2
- net at R2.1, R5.2, U1.13 (-): now also C1.1
- net at R1.1, R6.2, U1.2 (-): now also C2.1
- new net: D1.2 (A), J11.1 (+12V)
- new net: D2.1 (K), J11.4 (-12V)
