File: 4u-variable-integrator/kicad/power.kicad_sch (KiCad schematic)
At the start: 16 parts, among them J17 4U_Power, U1 TL074, U2 LM13700, U4 TL072

Commit message: Refreshing kicad projects
Parts:
- removed C10, C5, C6, C7, C8, C9: 100nF, rumblesan-standard-parts:C_Rect_L7.0mm_W3.5mm_P5.00mm, symbol Device:C
- removed C11, C12: 1uF, rumblesan-standard-parts:CP_Radial_D5.0mm_P2.00mm, symbol Device:C_Polarized
- removed D3, D4: 1N5818, rumblesan-standard-parts:D_DO-41_SOD81_P10.16mm_Horizontal, symbol Diode:1N5818
- removed J17: 4U_Power, 4u-power:4u_Power_Molex_KK-254_P2.54mm, symbol 4U_Hardware:4U_Power
- removed R19: 1k, rumblesan-standard-parts:R_Axial_DIN0207_L6.3mm_D2.5mm_P10.16mm_Horizontal, symbol rumblesan-standard-parts:R
- added C10, C5, C6, C7, C8, C9: 100nF, Rumblesan_Standard_Parts:C_Rect_L7.0mm_W3.5mm_P5.00mm, symbol Rumblesan Standard Parts:C
- added C11, C12: 10uF, Rumblesan_Standard_Parts:CP_Radial_D5.0mm_P2.00mm, symbol Rumblesan Standard Parts:C_Polarized
- added D3, D4: 1N5818, Rumblesan_Standard_Parts:D_DO-41_SOD81_P10.16mm_Horizontal, symbol Device:D_Schottky
- added J17: 4U_Power, 4U_Power:4u_Power_Molex_KK-254_P2.54mm, symbol 4U_Power:4U_Power
- added R19: 1k, Rumblesan_Standard_Parts:R_Axial_DIN0207_L6.3mm_D2.5mm_P10.16mm_Horizontal, symbol Rumblesan Standard Parts:R
- D5: footprint rumblesan-standard-parts:D_DO-35_SOD27_P7.62mm_Horizontal -> Rumblesan_Standard_Parts:D_DO-35_SOD27_P7.62mm_Horizontal
- U1: footprint rumblesan-standard-parts:DIP-14_W7.62mm_Socket -> Rumblesan_Standard_Parts:DIP-14_W7.62mm_Socket
- U2: footprint rumblesan-standard-parts:DIP-16_W7.62mm_Socket -> Rumblesan_Standard_Parts:DIP-16_W7.62mm_Socket
- U4: footprint rumblesan-standard-parts:DIP-8_W7.62mm_Socket -> Rumblesan_Standard_Parts:DIP-8_W7.62mm_Socket
Connections:
- net +12V: now also C11.1, C5.1, C7.1, C9.1, D3.1 (K), R19.2
- net -12V: now also C10.2, C12.2, C6.2, C8.2, D4.2 (A)
- net GND: now also C10.1, C11.2, C12.1, C5.2, C6.1, C7.2, C8.1, C9.2, J17.2 (GND), J17.3 (GND)
- net V_REF: now also R19.1
- new net: D3.2 (A), J17.1 (+12V)
- new net: D4.1 (K), J17.4 (-12V)
