File: 4u-variable-integrator/kicad/4u-variable-integrator.kicad_sch (KiCad schematic)
At the start: 52 parts, among them J1 Banana Socket PanelMount, J10 Banana Socket PanelMount, J11 Banana Socket PanelMount, J12 Conn_01x04_Female, J13 Conn_01x04_Male, J14 Conn_01x02_Female, J15 Conn_01x02_Male, J16 Banana Socket PanelMount, J2 Banana Socket PanelMount, J3 Banana Socket PanelMount, J4 Conn_01x04_Female, J5 Conn_01x04_Female, J6 Conn_01x04_Male, J7 Conn_01x04_Male, J8 Banana Socket PanelMount, J9 Banana Socket PanelMount, Q1 2N3906, Q2 2N3906, U1 TL074, U2 LM13700

Commit message: Refreshing kicad projects
Parts:
- removed C1, C3: 100pF, rumblesan-standard-parts:C_Rect_L7.0mm_W3.5mm_P5.00mm, symbol Device:C
- removed C2, C4: 1nF, rumblesan-standard-parts:C_Rect_L7.0mm_W3.5mm_P5.00mm, symbol Device:C
- added C1, C3: 100pF, Rumblesan_Standard_Parts:C_Rect_L7.0mm_W3.5mm_P5.00mm, symbol Rumblesan Standard Parts:C
- added C2, C4: 1nF, Rumblesan_Standard_Parts:C_Rect_L7.0mm_W3.5mm_P5.00mm, symbol Rumblesan Standard Parts:C
- D1, D2: value 1n4148 -> 1N4148; footprint rumblesan-standard-parts:D_DO-35_SOD27_P7.62mm_Horizontal -> Rumblesan_Standard_Parts:D_DO-35_SOD27_P7.62mm_Horizontal
- H1, H2, H3, H4: footprint rumblesan-standard-parts:MountingHole_3.2mm_M3_DIN965_Pad -> Rumblesan_Standard_Parts:MountingHole_3.2mm_M3_DIN965_Pad
- J1, J10, J11, J16, J2, J3, J8, J9: footprint rumblesan-standard-parts:BananaJack_THT_JohnsonCinch_108-09 -> Rumblesan_Standard_Parts:BananaJack_THT_JohnsonCinch_108-09; symbol BananaJacks:Banana Socket PanelMount -> Banana_Jacks:Banana_Socket_PanelMount
- J12, J4, J5: symbol Connector:Conn_01x04_Female -> Connector:Conn_01x04_Socket
- J13, J6, J7: symbol Connector:Conn_01x04_Male -> Connector:Conn_01x04_Pin
- J14: symbol Connector:Conn_01x02_Female -> Connector:Conn_01x02_Socket
- J15: symbol Connector:Conn_01x02_Male -> Connector:Conn_01x02_Pin
- R1, R10, R11, R12, R13, R14, R15, R16, R17, R18, R2, R3, R4, R5, R6, R7, R8, R9: footprint rumblesan-standard-parts:R_Axial_DIN0207_L6.3mm_D2.5mm_P10.16mm_Horizontal -> Rumblesan_Standard_Parts:R_Axial_DIN0207_L6.3mm_D2.5mm_P10.16mm_Horizontal; symbol rumblesan-standard-parts:R -> Rumblesan Standard Parts:R
- RV1, RV2, RV3, RV4: footprint rumblesan-standard-parts:Potentiometer_Alpha_RD901F-40-00D_Single_Vertical -> Rumblesan_Standard_Parts:Potentiometer_Alpha_RD901F-40-00D_Single_Vertical
- U1: footprint rumblesan-standard-parts:DIP-14_W7.62mm_Socket -> Rumblesan_Standard_Parts:DIP-14_W7.62mm_Socket
- U2: footprint rumblesan-standard-parts:DIP-16_W7.62mm_Socket -> Rumblesan_Standard_Parts:DIP-16_W7.62mm_Socket
Connections:
- net at U1.2 (-), U2.12: now also C2.1
- net at R9.2, U1.1: now also C2.2
- net at D1.1 (K), R4.1, R5.2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: now also C1.1
- net at D2.2 (A), Q2.2 (B), U1.8: now also C3.2
- net at D2.1 (K), R13.1, R14.2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: now also C3.1
- net at D1.2 (A), Q1.2 (B), U1.7: now also C1.2
- net at U1.13 (-), U2.5: now also C4.1
- net at R18.2, U1.14: now also C4.2

Commit message: Adding BOM info
Parts:
- H1, H2, H3, H4: now left out of the parts list
Changed lines of the file:
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@@
   )
   (symbol (lib_id "Mechanical:MountingHole_Pad") (at 81.28 182.88 0) (unit 1)
-    (in_bom yes) (on_board yes) (dnp no) (fields_autoplaced)
+    (in_bom no) (on_board yes) (dnp no) (fields_autoplaced)
     (property "Reference" "H1" (at 83.82 180.7015 0)
       (effects (font (size 1.27 1.27)) (justify left) hide)
@@
   )
   (symbol (lib_id "Mechanical:MountingHole_Pad") (at 91.44 182.88 0) (unit 1)
-    (in_bom yes) (on_board yes) (dnp no) (fields_autoplaced)
+    (in_bom no) (on_board yes) (dnp no) (fields_autoplaced)
     (property "Reference" "H3" (at 93.98 180.7015 0)
       (effects (font (size 1.27 1.27)) (justify left) hide)
@@
   )
   (symbol (lib_id "Mechanical:MountingHole_Pad") (at 96.52 182.88 0) (unit 1)
-    (in_bom yes) (on_board yes) (dnp no) (fields_autoplaced)
+    (in_bom no) (on_board yes) (dnp no) (fields_autoplaced)
     (property "Reference" "H4" (at 99.06 180.7015 0)
       (effects (font (size 1.27 1.27)) (justify left) hide)
@@
   )
   (symbol (lib_id "Mechanical:MountingHole_Pad") (at 86.36 182.88 0) (unit 1)
-    (in_bom yes) (on_board yes) (dnp no) (fields_autoplaced)
+    (in_bom no) (on_board yes) (dnp no) (fields_autoplaced)
     (property "Reference" "H2" (at 88.9 180.7015 0)
       (effects (font (size 1.27 1.27)) (justify left) hide)
